File: nanoshield.kicad_sch (KiCad schematic)
At the start: 40 parts, among them J1 Conn_01x02, J10 Conn_01x02, J11 Conn_01x05_Female, J2 Analog, J20 Conn_01x03, J3 Digital, J30 Conn_01x03, J31 Conn_01x03, J40 Conn_01x03, J41 Conn_01x03, J50 Conn_01x03, J51 Conn_01x03, J60 Conn_01x02, Q40 IRLML0030, Q41 IRLML0030, Q60 IRLML0030

Commit message: Added Pages
Parts:
- removed C1: 470uF, Capacitor_THT:CP_Radial_D10.0mm_P5.00mm, symbol Device:C
- removed J1: Conn_01x02, Connector_Phoenix_MC:PhoenixContact_MCV_1,5_2-G-3.5_1x02_P3.50mm_Vertical, symbol Connector_Generic:Conn_01x02
Other:
- added sheet Pi (Pi.kicad_sch)
- added sheet Power (Power.kicad_sch)
- note removed: "Voltage Input"
Changed lines of the file:
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@@
     (date "sam. 04 avril 2015")
   )
-  (junction (at 43.18 33.02) (diameter 0) (color 0 0 0 0)
-  )
   (junction (at 128.27 49.53) (diameter 0) (color 0 0 0 0)
   )
@@
   (junction (at 245.11 111.76) (diameter 0) (color 0 0 0 0)
   )
-  (junction (at 43.18 45.72) (diameter 0) (color 0 0 0 0)
-  )
   (junction (at 111.76 39.37) (diameter 0) (color 0 0 0 0)
   )
@@
     (stroke (width 0) (type default) (color 0 0 0 0))
   )
-  (wire (pts (xy 43.18 40.64) (xy 43.18 45.72))
-    (stroke (width 0) (type default) (color 0 0 0 0))
-  )
   (wire (pts (xy 33.02 86.36) (xy 33.02 125.73))
     (stroke (width 0) (type solid) (color 0 0 0 0))
@@
     (stroke (width 0) (type default) (color 0 0 0 0))
   )
-  (wire (pts (xy 54.61 33.02) (xy 54.61 35.56))
-    (stroke (width 0) (type default) (color 0 0 0 0))
-  )
   (wire (pts (xy 60.96 102.87) (xy 76.2 102.87))
     (stroke (width 0) (type solid) (color 0 0 0 0))
@@
     (stroke (width 0) (type default) (color 0 0 0 0))
   )
-  (wire (pts (xy 54.61 45.72) (xy 43.18 45.72))
-    (stroke (width 0) (type default) (color 0 0 0 0))
-  )
   (wire (pts (xy 254 33.02) (xy 254 35.56))
     (stroke (width 0) (type default) (color 0 0 0 0))
@@
     (stroke (width 0) (type default) (color 0 0 0 0))
   )
-  (wire (pts (xy 43.18 33.02) (xy 43.18 38.1))
-    (stroke (width 0) (type default) (color 0 0 0 0))
-  )
-  (wire (pts (xy 54.61 43.18) (xy 54.61 45.72))
-    (stroke (width 0) (type default) (color 0 0 0 0))
-  )
   (wire (pts (xy 22.86 120.65) (xy 40.64 120.65))
     (stroke (width 0) (type solid) (color 0 0 0 0))
@@
     (stroke (width 0) (type default) (color 0 0 0 0))
   )
-  (wire (pts (xy 43.18 31.75) (xy 43.18 33.02))
-    (stroke (width 0) (type default) (color 0 0 0 0))
-  )
   (wire (pts (xy 261.62 111.76) (xy 245.11 111.76))
     (stroke (width 0) (type default) (color 0 0 0 0))
@@
     (stroke (width 0) (type default) (color 0 0 0 0))
   )
-  (wire (pts (xy 43.18 45.72) (xy 43.18 46.99))
-    (stroke (width 0) (type default) (color 0 0 0 0))
-  )
   (wire (pts (xy 63.5 118.11) (xy 63.5 128.27))
     (stroke (width 0) (type solid) (color 0 0 0 0))
@@
     (stroke (width 0) (type default) (color 0 0 0 0))
   )
-  (wire (pts (xy 43.18 33.02) (xy 54.61 33.02))
-    (stroke (width 0) (type default) (color 0 0 0 0))
-  )
   (wire (pts (xy 38.1 123.19) (xy 38.1 128.27))
     (stroke (width 0) (type solid) (color 0 0 0 0))
@@
   )
   (text "Digital-Ausgang 2" (at 246.38 86.36 0)
-    (effects (font (size 1.27 1.27)) (justify left bottom))
-  )
-  (text "Voltage Input" (at 35.56 25.4 0)
     (effects (font (size 1.27 1.27)) (justify left bottom))
   )
@@
     (pin "2")
   )
-  (symbol (lib_name "VCC_9") (lib_id "power:VCC") (at 43.18 31.75 0) (mirror y) (unit 1)
-    (in_bom yes) (on_board yes) (fields_autoplaced)
-    (property "Reference" "#PWR01" (id 0) (at 43.18 35.56 0)
-      (effects (font (size 1.27 1.27)) hide)
-    )
-    (property "Value" "VCC" (id 1) (at 43.18 26.67 0))
-    (property "Footprint" "" (id 2) (at 43.18 31.75 0)
-      (effects (font (size 1.27 1.27)) hide)
-    )
-    (property "Datasheet" "" (id 3) (at 43.18 31.75 0)
-      (effects (font (size 1.27 1.27)) hide)
-    )
-    (pin "1")
-  )
   (symbol (lib_id "power:GND") (at 24.13 190.5 0) (unit 1)
     (in_bom yes) (on_board yes) (fields_autoplaced)
@@
     (pin "2")
     (pin "3")
-  )
-  (symbol (lib_name "GND_4") (lib_id "power:GND") (at 43.18 46.99 0) (mirror y) (unit 1)
-    (in_bom yes) (on_board yes)
-    (property "Reference" "#PWR02" (id 0) (at 43.18 53.34 0)
-      (effects (font (size 1.27 1.27)) hide)
-    )
-    (property "Value" "GND" (id 1) (at 43.18 50.8 0))
-    (property "Footprint" "" (id 2) (at 43.18 46.99 0)
-      (effects (font (size 1.27 1.27)) hide)
-    )
-    (property "Datasheet" "" (id 3) (at 43.18 46.99 0)
-      (effects (font (size 1.27 1.27)) hide)
-    )
-    (pin "1")
-  )
-  (symbol (lib_id "Connector_Generic:Conn_01x02") (at 38.1 38.1 0) (mirror y) (unit 1)
-    (in_bom yes) (on_board yes) (fields_autoplaced)
-    (property "Reference" "J1" (id 0) (at 35.56 38.0999 0)
-      (effects (font (size 1.27 1.27)) (justify left))
-    )
-    (property "Value" "Conn_01x02" (id 1) (at 35.56 40.6399 0)
-      (effects (font (size 1.27 1.27)) (justify left))
-    )
-    (property "Footprint" "Connector_Phoenix_MC:PhoenixContact_MCV_1,5_2-G-3.5_1x02_P3.50mm_Vertical" (id 2) (at 38.1 38.1 0)
-      (effects (font (size 1.27 1.27)) hide)
-    )
-    (property "Datasheet" "~" (id 3) (at 38.1 38.1 0)
-      (effects (font (size 1.27 1.27)) hide)
-    )
-    (pin "1")
-    (pin "2")
   )
   (symbol (lib_id "Connector_Generic:Conn_01x03") (at 264.16 146.05 0) (unit 1)
@@
     (pin "2")
   )
-  (symbol (lib_id "Device:C") (at 54.61 39.37 0) (unit 1)
-    (in_bom yes) (on_board yes)
-    (property "Reference" "C1" (id 0) (at 58.42 38.0999 0)
-      (effects (font (size 1.27 1.27)) (justify left))
-    )
-    (property "Value" "470uF" (id 1) (at 58.42 40.6399 0)
-      (effects (font (size 1.27 1.27)) (justify left))
-    )
-    (property "Footprint" "Capacitor_THT:CP_Radial_D10.0mm_P5.00mm" (id 2) (at 55.5752 43.18 0)
-      (effects (font (size 1.27 1.27)) hide)
-    )
-    (property "Datasheet" "~" (id 3) (at 54.61 39.37 0)
-      (effects (font (size 1.27 1.27)) hide)
-    )
-    (pin "1")
-    (pin "2")
-  )
   (symbol (lib_id "power:VCC") (at 92.71 27.94 0) (unit 1)
     (in_bom yes) (on_board yes) (fields_autoplaced)
@@
     (pin "3")
   )
+  (sheet (at 53.34 16.51) (size 25.4 8.89) (fields_autoplaced)
+    (stroke (width 0.1524) (type solid) (color 0 0 0 0))
+    (fill (color 0 0 0 0.0000))
+    (property "Sheet name" "Pi" (id 0) (at 53.34 15.7984 0)
+      (effects (font (size 1.27 1.27)) (justify left bottom))
+    )
+    (property "Sheet file" "Pi.kicad_sch" (id 1) (at 53.34 25.9846 0)
+      (effects (font (size 1.27 1.27)) (justify left top))
+    )
+  )
+  (sheet (at 19.05 19.05) (size 12.7 6.35) (fields_autoplaced)
+    (stroke (width 0.1524) (type solid) (color 0 0 0 0))
+    (fill (color 0 0 0 0.0000))
+    (property "Sheet name" "Power" (id 0) (at 19.05 18.3384 0)
+      (effects (font (size 1.27 1.27)) (justify left bottom))
+    )
+    (property "Sheet file" "Power.kicad_sch" (id 1) (at 19.05 25.9846 0)
+      (effects (font (size 1.27 1.27)) (justify left top))
+    )
+  )
   (sheet_instances
     (path "/" (page "1"))
+    (path "/f4aa7aa9-530a-4e7c-b9fe-6fc30ea153e5" (page "2"))
+    (path "/05fe5ca1-4a89-48a6-89a0-f0ba05481495" (page "3"))
   )
   (symbol_instances
-    (path "/7aa447b6-4b2a-48b9-96f8-5b03c91aed77"
-      (reference "#PWR01") (unit 1) (value "VCC") (footprint "")
-    )
-    (path "/81a57918-4be1-4e41-9702-ade84abbea83"
-      (reference "#PWR02") (unit 1) (value "GND") (footprint "")
-    )
     (path "/b454122d-badd-49fc-84df-a93057dd8dd7"
       (reference "#PWR03") (unit 1) (value "+5V") (footprint "")
@@
       (reference "#PWR0109") (unit 1) (value "GND") (footprint "")
     )
-    (path "/c691b4ee-27c9-4d6e-98cc-a89163c42868"
-      (reference "C1") (unit 1) (value "470uF") (footprint "Capacitor_THT:CP_Radial_D10.0mm_P5.00mm")
+    (path "/f4aa7aa9-530a-4e7c-b9fe-6fc30ea153e5/38244fe5-4108-406f-b745-c76097fc0b70"
+      (reference "#PWR?") (unit 1) (value "GND") (footprint "")
+    )
+    (path "/f4aa7aa9-530a-4e7c-b9fe-6fc30ea153e5/79250050-5353-499c-9492-eb93050d0382"
+      (reference "#PWR?") (unit 1) (value "VCC") (footprint "")
+    )
+    (path "/f4aa7aa9-530a-4e7c-b9fe-6fc30ea153e5/d4763eed-28ba-408f-b5e0-8ef31f5fb3f2"
+      (reference "#PWR?") (unit 1) (value "+5V") (footprint "")
+    )
+    (path "/f4aa7aa9-530a-4e7c-b9fe-6fc30ea153e5/ff0c8bff-4c09-4f4c-8a9c-6a274a78897a"
+      (reference "#PWR?") (unit 1) (value "+12V") (footprint "")
     )
     (path "/6bb35b3b-fcb5-4221-9b31-04ae7d4d482c"
@@
       (reference "C51") (unit 1) (value "0,47uF") (footprint "Capacitor_THT:C_Rect_L7.2mm_W3.0mm_P5.00mm_FKS2_FKP2_MKS2_MKP2")
     )
+    (path "/f4aa7aa9-530a-4e7c-b9fe-6fc30ea153e5/9e7b48b8-31ea-4a85-8206-eb5722e95333"
+      (reference "C?") (unit 1) (value "470uF") (footprint "Capacitor_THT:CP_Radial_D10.0mm_P5.00mm")
+    )
     (path "/583b9154-5b4f-4f54-a1e6-faec51164158"
       (reference "D10") (unit 1) (value "5,6V") (footprint "Diode_THT:D_DO-15_P12.70mm_Horizontal")
@@
       (reference "H2") (unit 1) (value "H2") (footprint "MountingHole:MountingHole_3.5mm_Pad")
     )
-    (path "/86e56b6b-ea36-457c-97cc-8f0150ba70ff"
-      (reference "J1") (unit 1) (value "Conn_01x02") (footprint "Connector_Phoenix_MC:PhoenixContact_MCV_1,5_2-G-3.5_1x02_P3.50mm_Vertical")
-    )
     (path "/00000000-0000-0000-0000-000056d719df"
       (reference "J2") (unit 1) (value "Analog") (footprint "Connector_PinHeader_2.54mm:PinHeader_1x15_P2.54mm_Vertical")
@@
       (reference "J60") (unit 1) (value "Conn_01x02") (footprint "Connector_Phoenix_MC:PhoenixContact_MCV_1,5_2-G-3.5_1x02_P3.50mm_Vertical")
     )
+    (path "/f4aa7aa9-530a-4e7c-b9fe-6fc30ea153e5/0bf9689d-d27b-4687-8395-a81cfcf33547"
+      (reference "J?") (unit 1) (value "Conn_01x02") (footprint "Connector_Phoenix_MC:PhoenixContact_MCV_1,5_2-G-3.5_1x02_P3.50mm_Vertical")
+    )
     (path "/fa8976cd-4235-4ac6-960e-8fd36c333d9f"
